Commit message: new marker for great tracking accuracy

File: ugv_visual_servoing/data/urdf/aruco.urdf (robot description, URDF)
Before this commit: robot aruco, 1 links, 0 joints
Links:
- link simple_box_base_link: geometry collision box size=0.4 0.4 0.1; visual mesh filename=package://ugv_visual_servoing/data/meshes/aruco_full.dae
